File: hw/key_sounder.kicad_sch (KiCad schematic)
At the start: 28 parts, among them J1 Conn_Coaxial_Power, J2 Screw_Terminal_01x02, J4 Screw_Terminal_01x02, J5 TRS-JACK-KP, Q1 G01N20LE, U1 LM393DR, U3 KS1, U3 Key, U4 Sounder

Commit message: Schematic updates.
Parts:
- renumbered U3 to KEY-EXT, U3 to KS1, R14 to R_Loop
Connections:
- net GND: now also C3.2, C4.2, C5.2, C6.2, C7.2, J2.1 (Pin_1), J4.2 (Pin_2), R_Loop.1
- net KOB_KEY-: now also J5.TN, U1.1 (1OUT)
- net at C1.1, C2.1, D5.1 (K)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: no longer KS1.1 (KEY), U4.1 (SND)
- new net: KS1.1 (KEY), U4.1 (SND)
- new net: KS1.2 (KEY), U4.2 (SND)
- no-connect marks 0 -> 2
Other:
- note added: "1/4in Key/Paddle Jack (Same as ICOM IC-7300)"
- company: (none) -> AESilky
- title: (none) -> MuKOB - Device
- moved on the sheet: C1, C2, C3, C4, C5, C6, C7, D1, D3, D5, D6, J1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

Commit message: Finish KOB page. UI FFC on.
Parts:
- removed Key/Paddle: Stereo-Plug, symbol Connector_Audio:AudioPlug3
- added J-SP1: Key-Paddle, symbol Audio-Plug-TRS:SP-TRS
- added R15: DNP, Resistor_SMD:R_1206_3216Metric_Pad1.30x1.75mm_HandSolder, symbol Device:R_US
- added TP1, TP2, TP3, TP4, TP5: Test_Point_01, symbol Test_point_Jump:TP_01
- KEY-EXT, KS1, U4: now left out of the parts list
- U1: value LM393DR -> LM393ADR; footprint Package_DIP:DIP-8_W7.62mm -> Package_SO:SOIC-8_3.9x4.9mm_P1.27mm; DK_Detail_Page /product-detail/en/texas-instruments/LM393DR/296-1015-1-ND/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 -> /product-detail/en/texas-instruments/LM393ADR/296-1015-1-ND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; Digi-Key_PN 296-1015-1-ND -> 296-14605-1-ND; MPN LM393DR -> LM393ADR
Connections:
- net GND: now also J-SP1.3 (S), R15.1
- net KOB_KEY-: now also TP2.1 (Pin_1)
- net LOOP_STATE: now also TP1.1 (Pin_1)
- net OFFSET_REF_V: now also TP3.1 (Pin_1)
- net SNDR_EN: now also TP4.1 (Pin_1)
- net at D4.2 (A), R10.2, U1.3: now also R15.2, TP5.1 (Pin_1)
- net at KEY-EXT.1 (KEY), Paddle.1 (DOT): now also J-SP1.1 (T)
- net at Paddle.3 (DASH): now also J-SP1.2 (R)
Other:
- note added: "Extrnal - Not part of MuKOB"
- moved on the sheet: C1, C2, C3, C4, C5, C6, C7, D1, D3, D4, D5, D6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

Commit message: Change display backlight GPIO.
Parts:
- renumbered C2 to C19, C1 to C20, C3 to C21, C4 to C22, C5 to C23, C6 to C24, C7 to C25, D5 to D1, D6 to D2, D1 to D4, D4 to D5, J1 to J15, J4 to J16, J2 to J17, J5 to J18, KEY-EXT to KEY-EXT1, Paddle to Paddle1, Q1 to Q2, R14 to R13, R2 to R14, R3 to R15, R10 to R16, R15 to R17, R_Loop to R_Loop1, TP4 to TP2, TP5 to TP4, TP2 to TP5, U4 to U5, U1 to U6
Other:
- title: MuKOB - Device -> MuKOB - Key/Paddle & Sounder

Commit message: Schematic prior to pulling KOB interface to separate board.
Parts:
- renumbered C22 to C10, C23 to C11, C24 to C12, C25 to C13, C19 to C7, C20 to C8, C21 to C9, D4 to D1, D1 to D2, D5 to D3, D3 to D4, D2 to D5, J17 to J10, J18 to J11, J15 to J8, J16 to J9, Q2 to Q1, R15 to R2, R17 to R3, R14 to R4, R16 to R5, R13 to R6, TP3 to TP4, TP2 to TP5, TP1 to TP6, TP4 to TP7, TP5 to TP8, U6 to U4
