File: hw/MuKOB.kicad_sch (KiCad schematic)
At the start: 29 parts, among them J1 MicroSD-Socket w/Det, J2 Conn_01x03, J3 Conn_02x15_Odd_Even, J4 SER_COM, J5 Conn_01x07, J6 Conn_01x04, J7 Conn_01x30, SW1 RESET, U1 PicoW, U2 MCP23S08-E/SO, U3 MAX3221

Commit message: Audio on main page. KeySounder Intf on separate board. Switch matrix via Resistors.
Parts:
- removed R1: DNP, Resistor_SMD:R_0402_1005Metric, symbol Device:R
- added BZ2: Buzzer, symbol Device:Buzzer
- added C10, C11, C12, C7, C8, C9: 0.1uF, symbol Device:C_Small
- added C13: 10uF, Capacitor_SMD:C_0402_1005Metric, symbol Device:C
- added C27: 0.1uF, Capacitor_SMD:C_0402_1005Metric, symbol Device:C
- added C28, C29: 1uF, Capacitor_SMD:C_0603_1608Metric, symbol Device:C
- added C30, C31: 1u, Capacitor_SMD:C_0805_2012Metric, symbol Device:C
- added C32, C33: 100nF, symbol Device:C_Small
- added C34, C37: 47u, Capacitor_SMD:C_0805_2012Metric, symbol Device:C
- added C35, C36, C38: 100n, Capacitor_SMD:C_0402_1005Metric, symbol Device:C
- added J10: SPKR_L, symbol Connector_Generic:Conn_01x02
- added J11: SPKR_R, symbol Connector_Generic:Conn_01x02
- added J15: SJ-43516-SMT-TR, symbol Connector_Audio:AudioJack4_Ground_SwitchTR1
- added J8: KEY_SND_IF, symbol Connector_Generic:Conn_01x07
- added J9: DISP_TP_SPI, symbol Connector_Generic:Conn_01x14
- added JP3: Conn_01x02, symbol Connector_Generic:Conn_01x02
- added LS2: Speaker, symbol Device:Speaker
- added M_DISP1, M_DISP2, M_DISP3, M_DISP4, M_DISP5, M_DISP6, M_KSI1, M_KSI2, M_KSI3, M_KSI4: MountingHole, MountingHole:MountingHole_2.7mm_M2.5, symbol Mechanical:MountingHole
- added OP5: OP_A-B, Connector_PinHeader_1.00mm:PinHeader_1x03_P1.00mm_Vertical, symbol MuKOB:Option_A-B
- added Q1: 2N3904, Package_TO_SOT_THT:TO-92_Inline, symbol Transistor_BJT:2N3904
- added R1: DNP, symbol Device:R_US
- added R2, R20, R21, R22: 100K, Resistor_SMD:R_0402_1005Metric, symbol Device:R
- added R23, R24: 10k, symbol Device:R_Small
- added R25: 100k, symbol Device:R_Small
- added R26, R29: 220, Resistor_SMD:R_0402_1005Metric, symbol Device:R
- added R27, R30: 100, Resistor_SMD:R_0402_1005Metric, symbol Device:R
- added R28, R31: 1.8K, Resistor_SMD:R_0402_1005Metric, symbol Device:R
- added R3: 10k, symbol Device:R_US
- added R4: 47k, symbol Device:R_US
- added R5: 28k, symbol Device:R_US
- added R6: 6.8k, symbol Device:R_US
- added R7: 15k, symbol Device:R_US
- added RE1: RotaryEncoder_Switch, symbol Device:RotaryEncoder_Switch
- added SW2: UP, Button_Switch_SMD:SW_Push_1P1T_NO_Vertical_Wuerth_434133025816, symbol Switch:SW_Push
- added SW3: RT, Button_Switch_SMD:SW_Push_1P1T_NO_Vertical_Wuerth_434133025816, symbol Switch:SW_Push
- added SW4: DN, Button_Switch_SMD:SW_Push_1P1T_NO_Vertical_Wuerth_434133025816, symbol Switch:SW_Push
- added SW5: LF, Button_Switch_SMD:SW_Push_1P1T_NO_Vertical_Wuerth_434133025816, symbol Switch:SW_Push
- added SW6: EN, Button_Switch_SMD:SW_Push_1P1T_NO_Vertical_Wuerth_434133025816, symbol Switch:SW_Push
- added TP10, TP12, TP13, TP9: Test_Point_01, symbol Test_point_Jump:TP_01
- added U4: TLV70033_SOT23-5, Package_TO_SOT_SMD:SOT-23-5, symbol Regulator_Linear:TLV70033_SOT23-5
- added U8: TPA2012D2RTJT, QFN50P400X400X80-21N270X270, symbol MuKOB:TPA2012D2RTJT
- added U9: NC7WZ16P6X, Package_TO_SOT_SMD:SOT-363_SC-70-6, symbol RPi_Pico:NC7WZ16P6X
- J5: value Conn_01x07 -> SPI-0
- J6: value Conn_01x04 -> I2C-0
Connections:
- net +3.3V: now also C13.1, J8.2 (Pin_2), J9.1 (Pin_1), R2.2, R20.2, R21.2, R22.2, R3.1, U8.13 (PVDD), U8.3 (PVDD); no longer J3.15 (Pin_15), J3.16 (Pin_16), J7.15 (Pin_15), J7.16 (Pin_16)
- net +3.3VA: now also C27.1, C29.1, C36.1, R23.1, R24.1, U4.5 (OUT), U8.9 (AVDD), U9.5 (VCC)
- net AUD_IN: now also U1.32 (GPIO27_ADC1); no longer U1.31 (GPIO26_ADC0)
- net DISP_BL_LED: now also J9.8 (Pin_8); no longer U1.27 (GPIO21)
- net DISP_CS-: now also J5.7 (Pin_7), J9.3 (Pin_3)
- net DISP_D/C-: now also J5.6 (Pin_6), J9.5 (Pin_5)
- net DISP_MISO: now also J9.9 (Pin_9)
- net DISP_MOSI: now also J5.4 (Pin_4), J9.6 (Pin_6)
- net DISP_RST-: now also J5.5 (Pin_5), J9.4 (Pin_4)
- net DISP_SCK: now also J5.3 (Pin_3), U1.19 (GPIO14), J9.7 (Pin_7); no longer U1.14 (GPIO10)
- net EX_CS-: no longer OP2.3 (B)
- net EX_IRQ: no longer OP1.3 (B)
- net GND: now also BZ2.2 (+), C10.2, C11.2, C12.2, C13.2, C7.2, C8.2, C9.2, J8.1 (Pin_1), J8.4 (Pin_4), J9.2 (Pin_2), JP3.2 (Pin_2), R1.2, R4.1, R5.1, R6.1, R7.1, RE1.C, RE1.S2, SW6.2, U8.12 (PGND), U8.21 (EXP), U8.4 (PGND), U9.2 (GND); no longer J3.14 (Pin_14), J3.17 (Pin_17), J7.14 (Pin_14), J7.17 (Pin_17)
- net GNDA: now also C27.2, C28.2, C29.2, C35.2, C36.2, C38.2, J15.G, J15.R2, Q1.1 (E), R27.1, R28.1, R30.1, R31.1, U4.2 (GND), U8.17 (INR-), U8.18 (AGND), U8.19 (INL-)
- net KEY_PDL_DOT: now also U1.5 (GPIO3), J8.6 (Pin_6); no longer U1.25 (GPIO19)
- net PDL_DASH: now also U1.6 (GPIO4), J8.7 (Pin_7); no longer U1.26 (GPIO20)
- net RE_A: now also J3.15 (Pin_15), J6.3 (Pin_3), J7.15 (Pin_15), U1.9 (GPIO6), RE1.A; no longer J3.23 (Pin_23), J7.23 (Pin_23), U1.19 (GPIO14)
- net RE_B: now also J3.16 (Pin_16), J6.4 (Pin_4), J7.16 (Pin_16), U1.10 (GPIO7), RE1.B; no longer J3.24 (Pin_24), J7.24 (Pin_24), U1.20 (GPIO15)
- net RE_SW: now also J3.17 (Pin_17), J7.17 (Pin_17); no longer J3.25 (Pin_25), J7.25 (Pin_25), U1.29 (GPIO22)
- net SDD_TGR: now also U1.20 (GPIO15); no longer U1.34 (GPIO28_ADC2)
- net SD_CS-: now also U1.27 (GPIO21); no longer J3.22 (Pin_22), J7.22 (Pin_22), U1.7 (GPIO5)
- net SD_TP_EX_MISO: now also J3.13 (Pin_13), J7.13 (Pin_13), U1.21 (GPIO16), J9.13 (Pin_13); no longer U1.6 (GPIO4)
- net SD_TP_EX_MOSI: now also J3.12 (Pin_12), J7.12 (Pin_12), U1.25 (GPIO19), J9.12 (Pin_12); no longer U1.5 (GPIO3)
- net SD_TP_EX_SCK: now also J3.10 (Pin_10), J7.10 (Pin_10), U1.24 (GPIO18), J9.10 (Pin_10), R1.1; no longer U1.4 (GPIO2)
- net SNDR_EN: now also U1.4 (GPIO2), J8.5 (Pin_5); no longer U1.24 (GPIO18)
- net SP_SW1: no longer J6.4 (Pin_4), OP2.1 (A), U2.11 (GP1)
- net SP_SW2: no longer J6.3 (Pin_3), OP1.1 (A), U2.12 (GP2)
- net TCH_CS-: now also U1.22 (GPIO17), J9.11 (Pin_11); no longer J5.7 (Pin_7), U1.9 (GPIO6)
- net TCH_IRQ-: now also J3.14 (Pin_14), J7.14 (Pin_14), U1.26 (GPIO20), J9.14 (Pin_14); no longer J3.18 (Pin_18), J5.6 (Pin_6), J7.18 (Pin_18), U1.10 (GPIO7)
- net TONE_GEN_L: now also U1.29 (GPIO22), OP5.2 (C), TP12.1 (Pin_1); no longer U1.32 (GPIO27_ADC1)
- net VOL_A: now also R2.1, TP9.1 (Pin_1), U8.15 (G0)
- net VOL_B: now also R20.1, TP10.1 (Pin_1), U8.1 (G1)
- net VSYS: now also C28.1, J8.3 (Pin_3), U4.1 (IN), U4.3 (EN)
- net at OP2.2 (C): no longer U1.21 (GPIO16)
- net at OP1.2 (C): no longer U1.22 (GPIO17)
- net HAS_AUD: no longer names the net of U2.13 (GP3)
- net HAS_AUD: no longer TP11.1 (Pin_1)
- removed net SD_TCH_MISO: J3.13 (Pin_13), J3.20 (Pin_20), J5.5 (Pin_5), J7.13 (Pin_13), J7.20 (Pin_20)
- removed net SD_TCH_MOSI: J3.12 (Pin_12), J3.21 (Pin_21), J5.4 (Pin_4), J7.12 (Pin_12), J7.21 (Pin_21)
- removed net SD_TCH_SCK: J3.10 (Pin_10), J3.19 (Pin_19), J5.3 (Pin_3), J7.10 (Pin_10), J7.19 (Pin_19)
- net TONE_GEN_R renamed TONE_GEN_R_SPKR
- net TONE_GEN_R_SPKR: now also TP11.1 (Pin_1), U9.1 (A1)
- new net: C31.1, U8.16 (INR+)
- new net: C31.2, J15.R1N
- new net: JP3.1 (Pin_1), R21.1, U8.8 (~{SDR})
- new net: R4.2, SW2.2
- new net: C32.2, Q1.3 (C), R23.2, R25.1
- new net: R7.2, SW5.2
- new net: R22.1, U8.7 (~{SDL})
- new net: J11.1 (Pin_1), U8.14 (OUTR+)
- new net: J11.2 (Pin_2), U8.11 (OUTR-)
- new net: C33.1, Q1.2 (B), R25.2
- new net: J10.1 (Pin_1), U8.2 (OUTL+)
- new net: J10.2 (Pin_2), U8.5 (OUTL-)
- new net: R6.2, SW4.2
- new net: C30.2, J15.TN
- new net: C30.1, U8.20 (INL+)
- new net: R5.2, SW3.2
- new net: J3.18 (Pin_18), J7.18 (Pin_18)
- new net: J3.19 (Pin_19), J7.19 (Pin_19)
- new net: J3.20 (Pin_20), J7.20 (Pin_20)
- new net: J3.21 (Pin_21), J7.21 (Pin_21)
- new net: J3.22 (Pin_22), J7.22 (Pin_22)
- new net: J3.23 (Pin_23), J7.23 (Pin_23)
- new net: J3.24 (Pin_24), J7.24 (Pin_24)
- new net: J3.25 (Pin_25), J7.25 (Pin_25)
- new net BUZZ_DRV: BZ2.1 (-), OP5.1 (A)
- new net MIC: C32.1, TP13.1 (Pin_1)
- new net MIC_IN: C33.2, J15.S, R24.2
- new net PWM_AUD_L: C37.1, J15.T, R31.2
- new net PWM_AUD_R: C34.1, J15.R1, R28.2
- new net PWM_L: R29.2, U9.4 (Y2)
- new net PWM_LL: C37.2, C38.1, R29.1, R30.2
- new net PWM_R: R26.2, U9.6 (Y1)
- new net PWM_RR: C34.2, C35.1, R26.1, R27.2
- new net SW_MTRX: C10.1, C11.1, C12.1, C7.1, C8.1, C9.1, R3.2, RE1.S1, SW2.1, SW3.1, SW4.1, SW5.1, SW6.1, U1.31 (GPIO26_ADC0)
- new net TONE_GEN_L_SPKR: OP5.3 (B), U9.3 (A2)
- no-connect marks 8 -> 10
Other:
- removed sheet Audio
- removed sheet Key Sounder
- note added: "3.5mm TRRS Audio (STD)"
- note added: "Audio Output Option"
- note added: "Audio+ Option (requires IO Expansion for volume)"
- note added: "CS-"
- note added: "DC-"
- note added: "Mic input (optional)"
- note added: "Needed for Analog out and/or Mic in"
- note added: "OP4:1-2+BZ1 or OP4:2-3+rest"
- note added: "RES"
- note added: "SCL"
- note added: "SDA"
- note added: "SPI-OLED (Instead of TFT)"
- note removed: "SPI-0"
- note removed: "SPI0_CS-"
- note removed: "SPI0_DC-"
- note removed: "SPI0_RES"
- note removed: "SPI0_SCL"
- note removed: "SPI0_SDA"
- company: AESilky -> Silky-Design (AESilky)
- moved on the sheet: C2, C3, C4, C5, C6, J3, J4, J5, J7, JP1, M_H1, M_H2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
