File: hw/MuKOB.kicad_sch (KiCad schematic)
At the start: 99 parts, among them J1 MicroSD-Socket w/Det, J10 SPKR_L, J11 SPKR_R, J15 SJ-43516-SMT-TR, J2 Conn_01x03, J3 Conn_02x15_Odd_Even, J4 SER_COM, J5 SPI-0, J6 I2C-0, J7 Conn_01x30, J8 KEY_SND_IF, J9 DISP_TP_SPI, Q1 2N3904, SW1 RESET, SW2 UP, SW3 RT, SW4 DN, SW5 LF, SW6 EN, U1 PicoW, U2 MCP23S08-E/SO, U3 MAX3221, U4 TLV70033_SOT23-5, U8 TPA2012D2RTJT, U9 NC7WZ16P6X

Commit message: Reorganize onto 3 boards. Use 20pin UI connector.
Parts:
- removed J3: Conn_02x15_Odd_Even, symbol Connector_Generic:Conn_02x15_Odd_Even
- removed J7: Conn_01x30, symbol Connector_Generic:Conn_01x30
- removed OP3: OP_A-B, Connector_PinHeader_1.00mm:PinHeader_1x03_P1.00mm_Vertical, symbol MuKOB:Option_A-B
- removed R2, R20, R21, R22: 100K, Resistor_SMD:R_0402_1005Metric, symbol Device:R
- removed R23, R24: 10k, symbol Device:R_Small
- removed R25: 100k, symbol Device:R_Small
- removed R26, R29: 220, Resistor_SMD:R_0402_1005Metric, symbol Device:R
- removed R27, R30: 100, Resistor_SMD:R_0402_1005Metric, symbol Device:R
- removed R28, R31: 1.8K, Resistor_SMD:R_0402_1005Metric, symbol Device:R
- removed TP7 (x2): Test_Point_01, symbol Test_point_Jump:TP_01
- added J1: Conn_02x10_Odd_Even, symbol Connector_Generic:Conn_02x10_Odd_Even
- added J12, J6: Conn_01x03, symbol Connector_Generic:Conn_01x03
- added J13: IO_EX, symbol Connector_Generic:Conn_01x07
- added J2: Conn_01x20, symbol Connector_Generic:Conn_01x20
- added LED1: PWR, LED_THT:LED_D5.0mm, symbol Device:LED
- added OP4, OP5, OP6, OP7, OP8: OP_A-B, Connector_PinHeader_1.00mm:PinHeader_1x03_P1.00mm_Vertical, symbol MuKOB:Option_A-B
- added R2: 150, Resistor_THT:R_Axial_DIN0207_L6.3mm_D2.5mm_P10.16mm_Horizontal, symbol Device:R_Small_US
- added R20, R21, R22, R23, R26: 100k, symbol Device:R_US
- added R24, R25: 10k, symbol Device:R_US
- added R27, R30: 220, symbol Device:R_US
- added R28, R31: 100, symbol Device:R_US
- added R29, R32: 1.8k, symbol Device:R_US
- C1: value 10u -> 10uF
- renumbered J2 to J3, J8 to J5, J15 to J7, J9 to J8, J5 to J9, JP3 to JP2, OP5 to OP1, OP1 to OP2, OP2 to OP3
Connections:
- net MIC is gone; now on net AUD_IN: C32.1, TP13.1 (Pin_1)
- net SDD_TGR is gone; now on net SD_CARD_DET: U1.20 (GPIO15)
- net +3.3V: now also J5.3 (Pin_3), J1.19 (Pin_19), J1.2 (Pin_2), J2.19 (Pin_19), J2.2 (Pin_2), R2.1, R20.1, R21.1, R22.1, R23.1; no longer J5.2 (Pin_2)
- net +3.3VA: now also R24.1, R25.1
- net DISP_BL_LED: now also J1.8 (Pin_8), J2.8 (Pin_8)
- net DISP_CS-: now also U1.14 (GPIO10), J1.3 (Pin_3), J2.3 (Pin_3); no longer U1.12 (GPIO9)
- net DISP_D/C-: now also U1.7 (GPIO5), J1.5 (Pin_5), J2.5 (Pin_5); no longer U1.11 (GPIO8)
- net DISP_MISO: now also J1.9 (Pin_9), J2.9 (Pin_9)
- net DISP_MOSI: now also J1.6 (Pin_6), J2.6 (Pin_6)
- net DISP_RST-: now also J1.4 (Pin_4), J2.4 (Pin_4)
- net DISP_SCK: now also J1.7 (Pin_7), J2.7 (Pin_7)
- net GND: now also J5.2 (Pin_2), J1.1 (Pin_1), J1.20 (Pin_20), J12.1 (Pin_1), J13.1 (Pin_1), J2.1 (Pin_1), J2.20 (Pin_20), J6.1 (Pin_1), LED1.1 (K); no longer J5.4 (Pin_4), U1.42 (GND)
- net GNDA: now also J12.3 (Pin_3), R28.2, R29.2, R31.2, R32.2
- net MIC_IN: now also R25.2
- net PWM_AUD_L: now also R32.1
- net PWM_AUD_R: now also R29.1
- net PWM_L: now also R30.2
- net PWM_LL: now also R30.1, R31.1
- net PWM_R: now also R27.2
- net PWM_RR: now also R27.1, R28.1
- net RE_A: now also J1.15 (Pin_15), J2.15 (Pin_15)
- net RE_B: now also J1.16 (Pin_16), J2.16 (Pin_16)
- net SD_CARD_DET: no longer U2.10 (GP0)
- net SD_TP_EX_MISO: now also J1.13 (Pin_13), J2.13 (Pin_13)
- net SD_TP_EX_MOSI: now also J1.12 (Pin_12), J2.12 (Pin_12)
- net SD_TP_EX_SCK: now also J1.10 (Pin_10), J2.10 (Pin_10)
- net SW_MTRX: now also J1.17 (Pin_17), J2.17 (Pin_17)
- net TCH_CS-: now also J1.11 (Pin_11), J2.11 (Pin_11)
- net TCH_IRQ-: now also J1.14 (Pin_14), J2.14 (Pin_14)
- net TONE_GEN_R_SPKR: now also OP8.3 (B)
- net VSYS: now also J5.4 (Pin_4); no longer J5.3 (Pin_3)
- net IO28AD2_TGR: now reaches U1.34 (GPIO28_ADC2)
- net IO28AD2_TGR: now also OP8.2 (C)
- net at U2.17 (GP7): now also J13.7 (Pin_7)
- net at JP2.1 (Pin_1), U8.8 (~{SDR}): now also R22.2
- net at C32.2, Q1.3 (C): now also R24.2, R26.1
- net at U8.7 (~{SDL}): now also R23.2
- net at C33.1, Q1.2 (B): now also R26.2
- net EX_VOL_B: now reaches U2.11 (GP1)
- net EX_VOL_B: now also OP7.3 (B)
- net at U2.12 (GP2): now also J13.2 (Pin_2)
- net at U2.13 (GP3): now also J13.3 (Pin_3)
- net at U2.16 (GP6): now also J13.6 (Pin_6)
- net at OP2.1 (A): now also OP4.2 (C)
- net at OP2.2 (C): now also U1.11 (GPIO8)
- net P_VOL_A: now reaches OP2.3 (B)
- net P_VOL_A: now also OP6.1 (A)
- net at OP3.1 (A): now also OP5.2 (C)
- net at OP3.2 (C): now also U1.12 (GPIO9)
- net P_VOL_B: now reaches OP3.3 (B)
- net P_VOL_B: now also OP7.1 (A)
- net EX_CS- renamed U1TX_EXCS-
- net U1TX_EXCS-: now also OP4.3 (B)
- net EX_IRQ: no longer names the net of U2.8 (INT)
- net EX_IRQ: now also OP5.3 (B)
- net SWCLK: no longer names the net of U1.41 (SWCLK)
- net SWDIO: no longer names the net of U1.43 (SWDIO)
- net VOL_A renamed VOLA
- net VOLA: now also OP6.2 (C), R20.2; no longer U2.14 (GP4)
- net VOL_B renamed VOLB
- net VOLB: now also OP7.2 (C), R21.2; no longer U2.15 (GP5)
- new net: J13.4 (Pin_4), U2.14 (GP4)
- new net: J13.5 (Pin_5), U2.15 (GP5)
- new net: J1.18 (Pin_18), J2.18 (Pin_18)
- new net: LED1.2 (A), R2.2
- new net: J6.3 (Pin_3), OP4.1 (A)
- new net: J6.2 (Pin_2), OP5.1 (A)
- new net EX_VOL_A: OP6.3 (B), U2.10 (GP0)
- new net GPIO28ADC2: J12.2 (Pin_2), OP8.1 (A)
- no-connect marks 10 -> 11
Other:
- note added: "Audio+ Option"
- note added: "IO Expansion"
- note added: "Needed for Analog out and Mic in"
- note added: "RX"
- note added: "Remove JP1 to use 3.5V serial for debug"
- note added: "Serial-0 3.3V"
- note added: "Serial-1 3.3V"
- note added: "Speaker Amplifier w/volume (optional)"
- note added: "TX"
- note added: "UI FFC Connector"
- note removed: "Audio+ Option (requires IO Expansion for volume)"
- note removed: "IO Expansion (Required for full audio+ opt)"
- note removed: "Needed for Analog out and/or Mic in"
- note removed: "Serial 3.3V"
- note removed: "User Interface FFC Connector"
- moved on the sheet: BZ2, C1, C10, C11, C12, C2, C3, C4, C5, C6, C7, C8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

Commit message: Electrical checks complete.
Parts:
- removed M_KSI1, M_KSI2, M_KSI3, M_KSI4: MountingHole, MountingHole:MountingHole_2.7mm_M2.5, symbol Mechanical:MountingHole
- added M_KSI1, M_KSI2, M_KSI3, M_KSI4: MountingHole_Pad, symbol Mechanical:MountingHole_Pad
- R2: value 150 -> 100
- renumbered TP9 to TP3, TP10 to TP4, TP13 to TP5, TP11 to TP6, TP12 to TP7, U8 to U5
Connections:
- net +3.3V: now also J1.1 (Pin_1), J2.1 (Pin_1); no longer J1.2 (Pin_2), J2.2 (Pin_2)
- net GND: now also J1.2 (Pin_2), J2.2 (Pin_2), M_KSI1.1, M_KSI2.1, M_KSI3.1, M_KSI4.1; no longer J1.1 (Pin_1), J2.1 (Pin_1)
- net open18: now reaches J1.18 (Pin_18), J2.18 (Pin_18)
Other:
- note added: "IO Expansion Option"
- note added: "Serial Data Comm Option"
- note removed: "IO Expansion"
- note removed: "Serial Data Comm (Optional)"

Commit message: Schematic updates. Reorg components between boards. 20 pin ribbon.
Parts:
- removed J1: Conn_02x10_Odd_Even, symbol Connector_Generic:Conn_02x10_Odd_Even
- removed J8: DISP_TP_SPI, symbol Connector_Generic:Conn_01x14
- removed M_DISP4: MountingHole, MountingHole:MountingHole_2.7mm_M2.5, symbol Mechanical:MountingHole
- added J-SP1: Key-Paddle, symbol Audio-Plug-TRS:SP-TRS
- added J11: TRS-JACK-KP, symbol Connector_Audio:AudioJack3_SwitchT
- added J16: UI 20-Ribbon, symbol Connector_Generic:Conn_02x14_Odd_Even
- added KEY-EXT1: Key, symbol rpikobhat-rescue:Key-Telegraph
- added Paddle1: PDL_EXT, symbol Switch:SW_SPDT_MSM
- added R8: 2.2k, symbol Device:R_US
- M_DISP1: value MountingHole -> MountingHole-2_8
- M_DISP2: value MountingHole -> MountingHole-3_5
- M_DISP3: value MountingHole -> MountingHole-4_0
Connections:
- net open18 is gone; now on net GND: J2.18 (Pin_18)
- net +3.3V: now also J2.20 (Pin_20), J16.11 (Pin_11), J16.2 (Pin_2); no longer J2.19 (Pin_19)
- net DISP_BL_LED: now also J16.16 (Pin_16)
- net DISP_CS-: now also J16.6 (Pin_6)
- net DISP_D/C-: now also J16.10 (Pin_10)
- net DISP_MISO: now also J16.18 (Pin_18)
- net DISP_MOSI: now also J16.12 (Pin_12)
- net DISP_RST-: now also J16.8 (Pin_8)
- net DISP_SCK: now also J16.14 (Pin_14)
- net GND: now also J2.16 (Pin_16), J-SP1.3 (S), J11.S, J16.3 (Pin_3), J16.4 (Pin_4), J16.7 (Pin_7), KEY-EXT1.2 (KEY), Paddle1.2, R8.1; no longer J2.20 (Pin_20), SW6.2
- net KEY_PDL_DOT: now also J11.T; no longer J5.6 (Pin_6)
- net PDL_DASH: now also J11.R
- net RE_A: now also J16.1 (Pin_1)
- net RE_B: now also J2.17 (Pin_17), J16.5 (Pin_5); no longer J2.16 (Pin_16)
- net SD_TP_EX_MISO: now also J16.17 (Pin_17), J16.26 (Pin_26)
- net SD_TP_EX_MOSI: now also J16.15 (Pin_15), J16.24 (Pin_24)
- net SD_TP_EX_SCK: now also J16.20 (Pin_20)
- net SW_MTRX: now also J2.19 (Pin_19), J16.9 (Pin_9); no longer J2.17 (Pin_17)
- net TCH_CS-: now also J16.13 (Pin_13), J16.22 (Pin_22)
- net TCH_IRQ-: now also J16.19 (Pin_19), J16.28 (Pin_28)
- new net: J-SP1.1 (T), KEY-EXT1.1 (KEY), Paddle1.1
- new net: J-SP1.2 (R), Paddle1.3
- new net: R8.2, SW6.2
- new net KEY-: J11.TN, J5.6 (Pin_6)
Other:
- note added: "1/4in Key/Paddle Jack (Same as ICOM IC-7300)"
- note added: "Extrnal - Not part of MuKOB"
- note added: "UI 20-FFC"
- note removed: "UI FFC Connector"
- note removed: "UI RC"
- moved on the sheet: J2, J9, M_DISP5, M_DISP6

Commit message: Device (Main) and K&S-IF ready for layout.
Parts:
- removed C10, C11, C12, C7, C8, C9: 0.1uF, symbol Device:C_Small
- removed J11: TRS-JACK-KP, symbol Connector_Audio:AudioJack3_SwitchT
- removed J16: UI 20-Ribbon, symbol Connector_Generic:Conn_02x14_Odd_Even
- removed J2: Conn_01x20, symbol Connector_Generic:Conn_01x20
- removed J4: SER_COM, symbol Connector_Audio:AudioJack3
- removed J7: SJ-43516-SMT-TR, symbol Connector_Audio:AudioJack4_Ground_SwitchTR1
- removed R4: 47k, symbol Device:R_US
- removed R5: 28k, symbol Device:R_US
- removed R6: 6.8k, symbol Device:R_US
- removed R7: 15k, symbol Device:R_US
- removed R8: 2.2k, symbol Device:R_US
- added C21: 22uF Tant, Capacitor_Tantalum_SMD:CP_EIA-3528-15_AVX-H_Pad1.50x2.35mm_HandSolder, symbol Device:C_Polarized_Small_US
- added C22, C23, C24, C25, C26, C27: 0.1uF, Capacitor_SMD:C_0603_1608Metric_Pad1.08x0.95mm_HandSolder, symbol Device:C_Small
- added C7: 10uF, Capacitor_SMD:C_0603_1608Metric, symbol Device:C
- added J13: UI 20-RBN, Connector_PinHeader_2.54mm:PinHeader_2x10_P2.54mm_Vertical, symbol Connector_Generic:Conn_02x10_Odd_Even
- added J14: AUDIO, AES_Library:CUI_DEVICES_SJ43516_SMT-CPJ, symbol AES_Library:CUI_SJ-43516-SMT-4cCPJ
- added J16: SPI-DISP, Connector_PinSocket_2.54mm:PinSocket_1x14_P2.54mm_Vertical, symbol Connector_Generic:Conn_01x14
- added J17: SW_MATRIX, Connector_PinHeader_2.54mm:PinHeader_1x05_P2.54mm_Vertical, symbol Connector_Generic:Conn_01x05
- added J18: UIM 20-FCC, AES_Library:Amphenol_F51L_1x20_P1.00mm_Horizontal-FFC, symbol Connector_Generic:Conn_01x20
- added J19: UIM 20-RBN, Connector_PinHeader_2.54mm:PinHeader_2x10_P2.54mm_Vertical, symbol Connector_Generic:Conn_02x10_Odd_Even
- added J2: SERIAL-COMM, AES_Library:CUI_SJ-2524-SMT-TRS-audio-jack, symbol AES_Library:CUI_SJ-2524-SMT-TRS-tsw-audio-jack
- added J7: KEY-PADDLE, AES_Library:CUI_SJ-63063B-audio-jack, symbol AES_Library:CUI_SJ-63063B-14TRS-audio-jack
- added J9: UI 20-FCC, AES_Library:Amphenol_F51L_1x20_P1.00mm_Horizontal-FFC, symbol Connector_Generic:Conn_01x20
- added JP2: J7-BP, Connector_PinHeader_2.54mm:PinHeader_1x02_P2.54mm_Vertical, symbol Jumper:Jumper_2_Open
- added M_H5: Mount, MountingHole:MountingHole_3.2mm_M3_ISO7380, symbol Mechanical:MountingHole
- added OP9: DISP-BL-PWR, Connector_PinHeader_2.54mm:PinHeader_1x03_P2.54mm_Vertical, symbol MuKOB:Option_A-B
- added R17: 20k, Resistor_SMD:R_0402_1005Metric_Pad0.72x0.64mm_HandSolder, symbol Device:R_Small_US
- added R18: 100, Resistor_SMD:R_0402_1005Metric_Pad0.72x0.64mm_HandSolder, symbol Device:R_Small_US
- added R19: 47k, Resistor_SMD:R_0402_1005Metric_Pad0.72x0.64mm_HandSolder, symbol Device:R_US
- added R20: 15k, Resistor_SMD:R_0402_1005Metric_Pad0.72x0.64mm_HandSolder, symbol Device:R_US
- added R21: 2.2k, Resistor_SMD:R_0402_1005Metric_Pad0.72x0.64mm_HandSolder, symbol Device:R_US
- added R22: 28k, Resistor_SMD:R_0402_1005Metric_Pad0.72x0.64mm_HandSolder, symbol Device:R_US
- added R23: 6.8k, Resistor_SMD:R_0402_1005Metric_Pad0.72x0.64mm_HandSolder, symbol Device:R_US
- added SW7: DN, AES_Library:SW_PUSH_SMD_1P1T_NO_45x45mm-CK, symbol Switch:SW_Push
- added SW8: RE-AO, AES_Library:SW_PUSH_SMD_1P1T_NO_45x45mm-CK, symbol Switch:SW_Push
- added SW9: RE-BO, AES_Library:SW_PUSH_SMD_1P1T_NO_45x45mm-CK, symbol Switch:SW_Push
- BZ1: renamed from BZ2; footprint (none) -> Buzzer_Beeper:Buzzer_12x9.5RM7.6
- C1: renamed from C3; footprint (none) -> Capacitor_SMD:C_0603_1608Metric_Pad1.08x0.95mm_HandSolder
- C10: renamed from C28; footprint Capacitor_SMD:C_0603_1608Metric -> Capacitor_SMD:C_0201_0603Metric_Pad0.64x0.40mm_HandSolder
- C11: renamed from C29; footprint Capacitor_SMD:C_0603_1608Metric -> Capacitor_SMD:C_0201_0603Metric_Pad0.64x0.40mm_HandSolder
- C12: renamed from C30; value 1u -> 1uF; footprint Capacitor_SMD:C_0805_2012Metric -> Capacitor_SMD:C_0201_0603Metric_Pad0.64x0.40mm_HandSolder
- C13: renamed from C31; value 1u -> 1uF; footprint Capacitor_SMD:C_0805_2012Metric -> Capacitor_SMD:C_0201_0603Metric_Pad0.64x0.40mm_HandSolder
- C14: renamed from C32; footprint (none) -> Capacitor_SMD:C_0201_0603Metric_Pad0.64x0.40mm_HandSolder
- C15: renamed from C33; footprint (none) -> Capacitor_SMD:C_0201_0603Metric_Pad0.64x0.40mm_HandSolder
- C16: renamed from C34; value 47u -> 47uF; footprint Capacitor_SMD:C_0805_2012Metric -> Capacitor_SMD:C_1206_3216Metric_Pad1.33x1.80mm_HandSolder
- C17: renamed from C35; value 100n -> 100nF; footprint Capacitor_SMD:C_0402_1005Metric -> Capacitor_SMD:C_0201_0603Metric_Pad0.64x0.40mm_HandSolder
- C18: renamed from C36; value 100n -> 100nF; footprint Capacitor_SMD:C_0402_1005Metric -> Capacitor_SMD:C_0201_0603Metric_Pad0.64x0.40mm_HandSolder
- C19: renamed from C37; value 47u -> 47uF; footprint Capacitor_SMD:C_0805_2012Metric -> Capacitor_SMD:C_1206_3216Metric_Pad1.33x1.80mm_HandSolder
- C2, C6: footprint (none) -> Capacitor_SMD:C_0603_1608Metric_Pad1.08x0.95mm_HandSolder
- C20: renamed from C38; value 100n -> 100nF; footprint Capacitor_SMD:C_0402_1005Metric -> Capacitor_SMD:C_0201_0603Metric_Pad0.64x0.40mm_HandSolder
- C3: renamed from C5; footprint (none) -> Capacitor_SMD:C_0603_1608Metric_Pad1.08x0.95mm_HandSolder
- C5: renamed from C4; footprint (none) -> Capacitor_SMD:C_0603_1608Metric_Pad1.08x0.95mm_HandSolder
- C8: renamed from C13; footprint Capacitor_SMD:C_0402_1005Metric -> Capacitor_SMD:C_0603_1608Metric
- C9: renamed from C27; footprint Capacitor_SMD:C_0402_1005Metric -> Capacitor_SMD:C_0603_1608Metric_Pad1.08x0.95mm_HandSolder
- J1: renamed from J3; value Conn_01x03 -> UART0 IO01; footprint (none) -> Connector_PinHeader_2.54mm:PinHeader_1x03_P2.54mm_Vertical
- J10: renamed from J13; footprint (none) -> Connector_PinHeader_2.54mm:PinHeader_1x07_P2.54mm_Vertical
- J11: renamed from J10; footprint (none) -> TerminalBlock_Philmore:TerminalBlock_Philmore_TB132_1x02_P5.00mm_Horizontal
- J12: renamed from J11; footprint (none) -> TerminalBlock_Philmore:TerminalBlock_Philmore_TB132_1x02_P5.00mm_Horizontal
- J15: renamed from J9; footprint (none) -> Connector_PinHeader_2.54mm:PinHeader_1x07_P2.54mm_Vertical
- J3: renamed from J5; footprint (none) -> Connector_PinHeader_2.54mm:PinHeader_1x07_P2.54mm_Vertical
- J4: renamed from J12; value Conn_01x03 -> GPIO28; footprint (none) -> Connector_PinHeader_2.54mm:PinHeader_1x03_P2.54mm_Vertical
- J5: renamed from J6; footprint (none) -> Connector_PinSocket_2.54mm:PinSocket_1x04_P2.54mm_Vertical
- J6: renamed from J1; footprint Connector_Card:microSD_HC_Molex_104031-0811 -> AES_Library:SDCard-GCT_MEM2075-00-140-01-A
- J8: renamed from J6; value Conn_01x03 -> UART1 IO89; footprint (none) -> Connector_PinHeader_2.54mm:PinHeader_1x03_P2.54mm_Vertical
- JP1: value Conn_01x02 -> S0-RX; footprint (none) -> Connector_PinHeader_2.54mm:PinHeader_1x02_P2.54mm_Vertical
- JP3: renamed from JP2; value Conn_01x02 -> AUD-SDR-; footprint (none) -> Connector_PinHeader_2.54mm:PinHeader_1x02_P2.54mm_Vertical
- LED1: footprint LED_THT:LED_D5.0mm -> AES_Library:LED_SMD_SIDEVIEW_Harvatek
- LS1: renamed from LS2; now left out of the parts list
- M_DISP1: value MountingHole-2_8 -> Disp-2.8; footprint MountingHole:MountingHole_2.7mm_M2.5 -> MountingHole:MountingHole_3.2mm_M3
- M_DISP2: value MountingHole-3_5 -> Disp-3.5; footprint MountingHole:MountingHole_2.7mm_M2.5 -> MountingHole:MountingHole_3.2mm_M3
- M_DISP3: value MountingHole-4_0 -> Disp-4.0; footprint MountingHole:MountingHole_2.7mm_M2.5 -> MountingHole:MountingHole_3.2mm_M3
- M_DISP4: renamed from M_DISP5; value MountingHole -> Mount
- M_DISP5: renamed from M_DISP6; value MountingHole -> Mount
- M_H1, M_H2, M_H3, M_H4: value MountingHole -> Mount; footprint MountingHole:MountingHole_2.7mm_M2.5 -> MountingHole:MountingHole_3.2mm_M3_ISO7380
- M_KSI1, M_KSI2, M_KSI3, M_KSI4: footprint (none) -> MountingHole:MountingHole_3.2mm_M3_ISO7380
- OP1: value OP_A-B -> BZ-SPK; footprint Connector_PinHeader_1.00mm:PinHeader_1x03_P1.00mm_Vertical -> Connector_PinHeader_2.54mm:PinHeader_1x03_P2.54mm_Vertical
- OP2, OP3, OP4, OP5, OP6, OP7: footprint Connector_PinHeader_1.00mm:PinHeader_1x03_P1.00mm_Vertical -> Connector_PinHeader_2.54mm:PinHeader_1x03_P2.54mm_Vertical
- OP8: value OP_A-B -> IO28-TR; footprint Connector_PinHeader_1.00mm:PinHeader_1x03_P1.00mm_Vertical -> Connector_PinHeader_2.54mm:PinHeader_1x03_P2.54mm_Vertical
- R1: renamed from R2; footprint Resistor_THT:R_Axial_DIN0207_L6.3mm_D2.5mm_P10.16mm_Horizontal -> Resistor_SMD:R_0402_1005Metric_Pad0.72x0.64mm_HandSolder
- R10: renamed from R26; footprint (none) -> Resistor_SMD:R_0402_1005Metric_Pad0.72x0.64mm_HandSolder
- R11: renamed from R27; footprint (none) -> Resistor_SMD:R_0402_1005Metric_Pad0.72x0.64mm_HandSolder
- R12: renamed from R28; footprint (none) -> Resistor_SMD:R_0402_1005Metric_Pad0.72x0.64mm_HandSolder
- R13: renamed from R29; footprint (none) -> Resistor_SMD:R_0402_1005Metric_Pad0.72x0.64mm_HandSolder
- R14: renamed from R30; footprint (none) -> Resistor_SMD:R_0402_1005Metric_Pad0.72x0.64mm_HandSolder
- R15: renamed from R31; footprint (none) -> Resistor_SMD:R_0402_1005Metric_Pad0.72x0.64mm_HandSolder
- R16: renamed from R32; footprint (none) -> Resistor_SMD:R_0402_1005Metric_Pad0.72x0.64mm_HandSolder
- R2: renamed from R1; footprint (none) -> Resistor_THT:R_Axial_DIN0207_L6.3mm_D2.5mm_P10.16mm_Horizontal
- R3: footprint (none) -> Resistor_SMD:R_0402_1005Metric_Pad0.72x0.64mm_HandSolder
- R4: renamed from R20; footprint (none) -> Resistor_SMD:R_0402_1005Metric_Pad0.72x0.64mm_HandSolder
- R5: renamed from R21; footprint (none) -> Resistor_SMD:R_0402_1005Metric_Pad0.72x0.64mm_HandSolder
- R6: renamed from R22; footprint (none) -> Resistor_SMD:R_0402_1005Metric_Pad0.72x0.64mm_HandSolder
- R7: renamed from R23; footprint (none) -> Resistor_SMD:R_0402_1005Metric_Pad0.72x0.64mm_HandSolder
- R8: renamed from R24; footprint (none) -> Resistor_SMD:R_0402_1005Metric_Pad0.72x0.64mm_HandSolder
- R9: renamed from R25; footprint (none) -> Resistor_SMD:R_0402_1005Metric_Pad0.72x0.64mm_HandSolder
- RE1: value RotaryEncoder_Switch -> RotEnc-SW; footprint (none) -> Rotary_Encoder:RotaryEncoder_Bourns_Vertical_PEC12R-3xxxF-Sxxxx
- SW1: footprint Button_Switch_SMD:SW_Push_1P1T_NO_Vertical_Wuerth_434133025816 -> AES_Library:SW_PUSH_SMD_1P1T_NO_45x45mm-CK
- SW2: value UP -> RE-SO; footprint Button_Switch_SMD:SW_Push_1P1T_NO_Vertical_Wuerth_434133025816 -> AES_Library:SW_PUSH_SMD_1P1T_NO_45x45mm-CK
- SW3: value RT -> UP; footprint Button_Switch_SMD:SW_Push_1P1T_NO_Vertical_Wuerth_434133025816 -> AES_Library:SW_PUSH_SMD_1P1T_NO_45x45mm-CK
- SW4: value DN -> LF; footprint Button_Switch_SMD:SW_Push_1P1T_NO_Vertical_Wuerth_434133025816 -> AES_Library:SW_PUSH_SMD_1P1T_NO_45x45mm-CK
- SW5: value LF -> EN; footprint Button_Switch_SMD:SW_Push_1P1T_NO_Vertical_Wuerth_434133025816 -> AES_Library:SW_PUSH_SMD_1P1T_NO_45x45mm-CK
- SW6: value EN -> RT; footprint Button_Switch_SMD:SW_Push_1P1T_NO_Vertical_Wuerth_434133025816 -> AES_Library:SW_PUSH_SMD_1P1T_NO_45x45mm-CK
- TP1: renamed from TP3; value Test_Point_01 -> VOL-A; footprint (none) -> Connector_PinSocket_2.54mm:PinSocket_1x01_P2.54mm_Vertical
- TP2: renamed from TP4; value Test_Point_01 -> VOL-B; footprint (none) -> Connector_PinSocket_2.54mm:PinSocket_1x01_P2.54mm_Vertical
- TP3: renamed from TP5; value Test_Point_01 -> AUD-IN; footprint (none) -> Connector_PinSocket_2.54mm:PinSocket_1x01_P2.54mm_Vertical
- TP4: renamed from TP6; value Test_Point_01 -> TONE-R; footprint (none) -> Connector_PinSocket_2.54mm:PinSocket_1x01_P2.54mm_Vertical
- TP5: renamed from TP7; value Test_Point_01 -> TONE-L; footprint (none) -> Connector_PinSocket_2.54mm:PinSocket_1x01_P2.54mm_Vertical
- U1: renamed from U3; footprint (none) -> AES_Library:TSSOP-16
- U2: renamed from U1; footprint RaspberryPI PicoW:RPi_PicoW_SMD_TH -> AES_Library:RPi_PicoW_SMD_TH
- U3: renamed from U2; footprint SOIC127P1030X265-18N -> Package_SO:SOIC-18W_7.5x11.6mm_P1.27mm
- U5: footprint QFN50P400X400X80-21N270X270 -> AES_Library:QFN50P400X400X80-21N270X270
- renumbered C1 to C4, U9 to U6
Connections:
- net +3.3V: now also C7.1, J13.11 (Pin_11), J13.2 (Pin_2), J16.1 (Pin_1), J18.1 (Pin_1), J18.20 (Pin_20), J19.11 (Pin_11), J19.2 (Pin_2), J9.1 (Pin_1), J9.20 (Pin_20), R17.1, R18.1
- net COM_RXD: now also J2.3
- net COM_TXD: now also J2.2
- net DISP_BL_LED: now also J13.16 (Pin_16), J16.8 (Pin_8), J18.8 (Pin_8), J19.16 (Pin_16), J9.8 (Pin_8), OP9.2 (C)
- net DISP_CS-: now also J13.6 (Pin_6), J16.3 (Pin_3), J18.3 (Pin_3), J19.6 (Pin_6), J9.3 (Pin_3)
- net DISP_D/C-: now also J13.10 (Pin_10), J16.5 (Pin_5), J18.5 (Pin_5), J19.10 (Pin_10), J9.5 (Pin_5)
- net DISP_MISO: now also J13.18 (Pin_18), J16.9 (Pin_9), J18.9 (Pin_9), J19.18 (Pin_18), J9.9 (Pin_9)
- net DISP_MOSI: now also J13.12 (Pin_12), J16.6 (Pin_6), J18.6 (Pin_6), J19.12 (Pin_12), J9.6 (Pin_6)
- net DISP_RST-: now also J13.8 (Pin_8), J16.4 (Pin_4), J18.4 (Pin_4), J19.8 (Pin_8), J9.4 (Pin_4)
- net DISP_SCK: now also J13.14 (Pin_14), J16.7 (Pin_7), J18.7 (Pin_7), J19.14 (Pin_14), J9.7 (Pin_7)
- net GND: now also RE1.S1, SW2.2, C21.2, C22.2, C23.2, C24.2, C25.2, C26.2, C27.2, C7.2, J13.3 (Pin_3), J13.4 (Pin_4), J13.7 (Pin_7), J16.2 (Pin_2), J17.2 (Pin_2), J17.5 (Pin_5), J18.16 (Pin_16), J18.18 (Pin_18), J18.2 (Pin_2), J19.3 (Pin_3), J19.4 (Pin_4), J19.7 (Pin_7), J2.1, J7.1, J9.16 (Pin_16), J9.18 (Pin_18), J9.2 (Pin_2), R19.1, R20.1, R21.1, R22.1, R23.1, SW8.2, SW9.2; no longer RE1.S2
- net GNDA: now also J14.4 (R2)
- net GPIO28ADC2: now also OP9.1 (A)
- net KEY-: now also J7.4, JP2.1 (A)
- net MIC_IN: now also J14.1 (S)
- net PWM_AUD_L: now also J14.2 (T)
- net PWM_AUD_R: now also J14.3 (R1)
- net RE_A: now also J13.1 (Pin_1), J17.1 (Pin_1), J18.15 (Pin_15), J19.1 (Pin_1), J9.15 (Pin_15), SW8.1
- net RE_B: now also J13.5 (Pin_5), J17.3 (Pin_3), J18.17 (Pin_17), J19.5 (Pin_5), J9.17 (Pin_17), SW9.1
- net RUN: now also C21.1, R17.2
- net SW_MTRX: now also RE1.S2, C22.1, C23.1, C24.1, C25.1, C26.1, C27.1, J13.9 (Pin_9), J17.4 (Pin_4), J18.19 (Pin_19), J19.9 (Pin_9), J9.19 (Pin_19), SW7.1; no longer RE1.S1
- net TCH_CS-: now also J13.19 (Pin_19), J16.11 (Pin_11), J18.11 (Pin_11), J19.19 (Pin_19), J9.11 (Pin_11)
- net TCH_IRQ-: now also J13.13 (Pin_13), J16.14 (Pin_14), J18.14 (Pin_14), J19.13 (Pin_13), J9.14 (Pin_14)
- net ExIO2: now reaches J10.2 (Pin_2), U3.12 (GP2)
- net ExIO3: now reaches J10.3 (Pin_3), U3.13 (GP3)
- net ExIO4: now reaches J10.4 (Pin_4), U3.14 (GP4)
- net ExIO5: now reaches J10.5 (Pin_5), U3.15 (GP5)
- net ExIO6: now reaches J10.6 (Pin_6), U3.16 (GP6)
- net ExIO7: now reaches J10.7 (Pin_7), U3.17 (GP7)
- net AIR+: now reaches C13.1, U5.16 (INR+)
- net at C13.2: now also J14.6 (R1N)
- net SDR-: now reaches JP3.1 (Pin_1), R6.2, U5.8 (~{SDR})
- net at SW5.2: now also R21.2
- net at SW6.2: now also R22.2
- net AOR+: now reaches J12.1 (Pin_1), U5.14 (OUTR+)
- net AOR-: now reaches J12.2 (Pin_2), U5.11 (OUTR-)
- net EX_INT: now reaches OP5.3 (B), U3.8 (INT)
- net AOL+: now reaches J11.1 (Pin_1), U5.2 (OUTL+)
- net AOL-: now reaches J11.2 (Pin_2), U5.5 (OUTL-)
- net at SW4.2: now also R20.2
- net at C12.2: now also J14.5 (TN)
- net AIL+: now reaches C12.1, U5.20 (INL+)
- net at SW3.2: now also R19.2
- net SDL-: now reaches R7.2, U5.7 (~{SDL})
- net EX_VOL_A renamed EX_VOLA
- net EX_VOL_B renamed EX_VOLB
- net IO28AD2_TGR renamed IO28_DBL_TGR
- net KEY_PDL_DOT renamed KEY_PDL_DOT-
- net KEY_PDL_DOT-: now also J7.2, JP2.2 (B)
- net PDL_DASH renamed PDL_DASH-
- net PDL_DASH-: now also J7.3
- net U1TX_EXCS- renamed EX_CS-
- new net: R23.2, SW7.2
- new net: OP9.3 (B), R18.2
- new net TCH_CLK: J13.20 (Pin_20), J16.10 (Pin_10), J18.10 (Pin_10), J19.20 (Pin_20), J9.10 (Pin_10)
- new net TCH_MISO: J13.15 (Pin_15), J16.13 (Pin_13), J18.13 (Pin_13), J19.15 (Pin_15), J9.13 (Pin_13)
- new net TCH_MOSI: J13.17 (Pin_17), J16.12 (Pin_12), J18.12 (Pin_12), J19.17 (Pin_17), J9.12 (Pin_12)
- no-connect marks 11 -> 12
Other:
- note added: "3.5mm TRRS Audio (Cell)"
- note added: "OP8:1-2+BZ1 or OP8:2-3+rest"
- note added: "Use when J7 not installed"
- note removed: "3.5mm TRRS Audio (STD)"
- note removed: "OP4:1-2+BZ1 or OP4:2-3+rest"
- note removed: "SPI-OLED (Instead of TFT)"
- note removed: "Serial-0 3.3V"
- note removed: "Serial-1 3.3V"
- note removed: "UI 20-FFC"
- moved on the sheet: BZ1, C12, C13, C14, C4, C8, C9, J11, J12, J15, J8, LED1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

Commit message: Main w/ UI - DRC close.
Parts:
- added CF1 (x10): 0.1uF, Capacitor_THT:C_Axial_L3.8mm_D2.6mm_P7.50mm_Horizontal, symbol Device:C_Small
- added JP-PWR-1, JP-PWR-2: PWR-APWR-Bridge, Connector_PinHeader_2.54mm:PinHeader_2x02_P2.54mm_Vertical, symbol Connector_Generic:Conn_02x02_Odd_Even
- M_KSI1, M_KSI2, M_KSI3, M_KSI4: footprint MountingHole:MountingHole_3.2mm_M3_ISO7380 -> MountingHole:MountingHole_3.2mm_M3_ISO7380_Pad_TopBottom
- OP8: value IO28-TR -> IO28-ToneR
Connections:
- net +3.3V: now also CF1.1, CF1.1, CF1.1, CF1.1, CF1.1, JP-PWR-1.3 (Pin_3), JP-PWR-2.3 (Pin_3); no longer J13.11 (Pin_11), J18.20 (Pin_20), J19.11 (Pin_11), J9.20 (Pin_20), R3.1
- net +3.3VA: now also J13.11 (Pin_11), J18.20 (Pin_20), J19.11 (Pin_11), J9.20 (Pin_20), R3.1, CF1.1, CF1.1, CF1.1, CF1.1, CF1.1, JP-PWR-1.4 (Pin_4), JP-PWR-2.4 (Pin_4)
- net GND: now also CF1.2, CF1.2, CF1.2, CF1.2, CF1.2, JP-PWR-1.1 (Pin_1), JP-PWR-2.1 (Pin_1); no longer C22.2, C23.2, C24.2, C25.2, C26.2, C27.2, J13.4 (Pin_4), J17.5 (Pin_5), J18.18 (Pin_18), J19.4 (Pin_4), J9.18 (Pin_18), R19.1, R20.1, R21.1, R22.1, R23.1, RE1.S1, SW2.2, SW8.2, SW9.2
- net GNDA: now also C22.2, C23.2, C24.2, C25.2, C26.2, C27.2, J13.4 (Pin_4), J17.5 (Pin_5), J18.18 (Pin_18), J19.4 (Pin_4), J9.18 (Pin_18), R19.1, R20.1, R21.1, R22.1, R23.1, RE1.S1, SW2.2, CF1.2, CF1.2, CF1.2, CF1.2, CF1.2, JP-PWR-1.2 (Pin_2), JP-PWR-2.2 (Pin_2)
- net KEY-: now also JP2.2 (B); no longer JP2.1 (A)
- net KEY_PDL_DOT-: now also JP2.1 (A); no longer JP2.2 (B)
- net GPIO08: now reaches OP2.2 (C), U2.11 (GPIO8)
- net GPIO09: now reaches OP3.2 (C), U2.12 (GPIO9)
- net U1TX_EXCS: now reaches OP2.1 (A), OP4.2 (C)
- net U1RX_EXINT: now reaches OP3.1 (A), OP5.2 (C)
- net U1_TX: now reaches J8.3 (Pin_3), OP4.1 (A)
- net U1_RX: now reaches J8.2 (Pin_2), OP5.1 (A)
- new net: SW8.2, SW9.2
Other:
- moved on the sheet: BZ1, C10, C11, C18, J15, J17, M_DISP4, M_DISP5, OP1, TP5, U4, U6

Commit message: Main PCB v1.0 complete.
Parts:
- renumbered CF1 to CF2, CF1 to CF3, CF1 to CF4, CF1 to CF5, CF1 to CFA1, CF1 to CFA2, CF1 to CFA3, CF1 to CFA4, CF1 to CFA5
Changed lines of the file:
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@@
     (fill (type none))
   )
-  (text_box "Jumper Settings:\n(All OP1-OP8:1-2 = Minimum Board)\n\nOP1:1-2 = BUZZER (No Audio)\n    2-3 = AUDIO (with Audio, with or w/o Amp)\n\nOP2,OP3,OP4,OP5:1-2 (no Audio Amp or ExpIO) =\n UART1 (GP 8&9) on J8\nWITH - Audio and Amp\nOP2,OP3:2-3 OP6,OP7:1-2 =\n Volume from Pico\nWITH - Expansion IO\nOP2,OP3:1-2 OP4,OP5:2-3 OP6,OP7:2-3 =\n Volume from Expansion IO (with Audio and Amp)\n ExGP2-7 available on J10\n\nOP8:1-2 = GP28/ADC2 to J4 & Display Backlight\n    2-3 = GP28 for Right Tone Gen\nOP9:1-2 = GP28/ADC2 Drives Display Backlight\n    2-3 = Fixed Display Backlight\nJP1: Closed for RS232 in\nOpen to use 3.3v (debug) Serial UART0"
+  (text_box "Jumper Settings:\n(All OP1-OP8:1-2 = Minimum Board)\n\nOP1:1-2 = BUZZER (No Audio)\n    2-3 = AUDIO (with Audio, with or w/o Amp)\n\nOP2,OP3,OP4,OP5:1-2 (no Audio Amp or ExpIO) =\n UART1 (GP 8&9) on J8\nWITH - Audio and Amp\nOP2,OP3:2-3 OP6,OP7:1-2 =\n Volume from Pico\nWITH - Expansion IO\nOP2,OP3:1-2 OP4,OP5:2-3 OP6,OP7:2-3 =\n Volume from Expansion IO (with Audio and Amp)\n ExGP2-7 available on J10\n\nOP8:1-2 = GP28/ADC2 to J4 & Display Backlight\n    2-3 = GP28 for Right Tone Gen\nOP9:1-2 = GP28/ADC2 Drives Display Backlight\n    2-3 = Fixed Display Backlight\nJP1: Closed for RS232 input\nOpen to use 3.3v (debug) Serial UART0"
     (at 335.28 12.7 0) (size 83.82 74.93)
     (stroke (width 0.8) (type default) (color 0 0 72 1))
@@
   (symbol (lib_id "Device:C_Small") (at 91.44 254 90) (unit 1)
     (in_bom yes) (on_board yes) (dnp no)
-    (property "Reference" "CF1" (at 90.17 252.73 90)
+    (property "Reference" "CF4" (at 90.17 252.73 90)
       (effects (font (size 1.27 1.27)) (justify left))
     )
@@
   (symbol (lib_id "Device:C_Small") (at 74.93 250.19 90) (unit 1)
     (in_bom yes) (on_board yes) (dnp no)
-    (property "Reference" "CF1" (at 73.66 248.92 90)
+    (property "Reference" "CFA1" (at 73.66 248.92 90)
       (effects (font (size 1.27 1.27)) (justify left))
     )
@@
   (symbol (lib_id "Device:C_Small") (at 58.42 254 90) (unit 1)
     (in_bom yes) (on_board yes) (dnp no)
-    (property "Reference" "CF1" (at 57.15 252.73 90)
+    (property "Reference" "CF2" (at 57.15 252.73 90)
       (effects (font (size 1.27 1.27)) (justify left))
     )
@@
   (symbol (lib_id "Device:C_Small") (at 107.95 257.81 90) (unit 1)
     (in_bom yes) (on_board yes) (dnp no)
-    (property "Reference" "CF1" (at 106.68 256.54 90)
+    (property "Reference" "CFA5" (at 106.68 256.54 90)
       (effects (font (size 1.27 1.27)) (justify left))
     )
@@
   (symbol (lib_id "Device:C_Small") (at 107.95 254 90) (unit 1)
     (in_bom yes) (on_board yes) (dnp no)
-    (property "Reference" "CF1" (at 106.68 252.73 90)
+    (property "Reference" "CFA4" (at 106.68 252.73 90)
       (effects (font (size 1.27 1.27)) (justify left))
     )
@@
   (symbol (lib_id "Device:C_Small") (at 74.93 257.81 90) (unit 1)
     (in_bom yes) (on_board yes) (dnp no)
-    (property "Reference" "CF1" (at 73.66 256.54 90)
+    (property "Reference" "CFA3" (at 73.66 256.54 90)
       (effects (font (size 1.27 1.27)) (justify left))
     )
@@
   (symbol (lib_id "Device:C_Small") (at 74.93 254 90) (unit 1)
     (in_bom yes) (on_board yes) (dnp no)
-    (property "Reference" "CF1" (at 73.66 252.73 90)
+    (property "Reference" "CFA2" (at 73.66 252.73 90)
       (effects (font (size 1.27 1.27)) (justify left))
     )
@@
   (symbol (lib_id "Device:C_Small") (at 58.42 257.81 90) (unit 1)
     (in_bom yes) (on_board yes) (dnp no)
-    (property "Reference" "CF1" (at 57.15 256.54 90)
+    (property "Reference" "CF3" (at 57.15 256.54 90)
       (effects (font (size 1.27 1.27)) (justify left))
     )
@@
   (symbol (lib_id "Device:C_Small") (at 91.44 257.81 90) (unit 1)
     (in_bom yes) (on_board yes) (dnp no)
-    (property "Reference" "CF1" (at 90.17 256.54 90)
+    (property "Reference" "CF5" (at 90.17 256.54 90)
       (effects (font (size 1.27 1.27)) (justify left))
     )
