File: hw/MK-KS-MkII.kicad_sch (KiCad schematic)
At the start: 62 parts, among them J10 KEY, J10 LOOP RES, J3 UART Data, J4 MuKOB IF, J7 KEY-PADDLE, J8 LOOP PWR, J9 SNDR/KOB, Q1 2N3904, Q1 G01N20LE, SW1 CLOSER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

Commit message: KSInf-MkIII: New  JA: Add terminal block
Parts:
- M_KSI1, M_KSI2, M_KSI3, M_KSI4, SHLD-1, SHLD-2, SHLD-3, SHLD-4: now left out of the parts list
- R2: value 100 -> 300
Other:
- moved on the sheet: SHLD-1, SHLD-2, SHLD-3, SHLD-4
Changed lines of the file:
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@@
 (kicad_sch (version 20230121) (generator eeschema)
-  (paper "B")
+  (paper "User" 419.1 323.85)
   (title_block
     (title "MuKOB - Key/Paddle & Sounder / MKOB USB Interface")
     (date "2024-01-16")
-    (rev "1")
+    (rev "1 B")
     (company "Silky-Design (AESilky)")
     (comment 1 "Copyright 2023-24 AESilky")
@@
   (junction (at 193.04 80.01) (diameter 0) (color 0 0 0 0)
   )
-  (junction (at 396.24 213.36) (diameter 0) (color 0 0 0 0)
+  (junction (at 27.94 274.32) (diameter 0) (color 0 0 0 0)
   )
   (junction (at 232.41 91.44) (diameter 0) (color 0 0 0 0)
@@
   (junction (at 172.72 231.14) (diameter 0) (color 0 0 0 0)
   )
-  (junction (at 396.24 218.44) (diameter 0) (color 0 0 0 0)
+  (junction (at 27.94 279.4) (diameter 0) (color 0 0 0 0)
   )
   (junction (at 165.1 64.77) (diameter 0) (color 0 0 0 0)
@@
   (junction (at 71.12 237.49) (diameter 0) (color 0 0 0 0)
   )
-  (junction (at 396.24 223.52) (diameter 0) (color 0 0 0 0)
+  (junction (at 27.94 284.48) (diameter 0) (color 0 0 0 0)
   )
   (junction (at 172.72 220.98) (diameter 0) (color 0 0 0 0)
@@
     (stroke (width 0) (type default))
   )
-  (wire (pts (xy 396.24 213.36) (xy 402.59 213.36))
+  (wire (pts (xy 27.94 274.32) (xy 34.29 274.32))
     (stroke (width 0) (type default))
   )
@@
     (stroke (width 0) (type default))
   )
-  (wire (pts (xy 396.24 213.36) (xy 396.24 218.44))
+  (wire (pts (xy 27.94 274.32) (xy 27.94 279.4))
     (stroke (width 0) (type default))
   )
@@
     (stroke (width 0) (type default))
   )
-  (wire (pts (xy 396.24 208.28) (xy 396.24 213.36))
+  (wire (pts (xy 27.94 269.24) (xy 27.94 274.32))
     (stroke (width 0) (type default))
   )
@@
     (stroke (width 0) (type default))
   )
-  (wire (pts (xy 396.24 223.52) (xy 402.59 223.52))
+  (wire (pts (xy 27.94 284.48) (xy 34.29 284.48))
     (stroke (width 0) (type default))
   )
@@
     (stroke (width 0) (type default))
   )
-  (wire (pts (xy 396.24 218.44) (xy 402.59 218.44))
+  (wire (pts (xy 27.94 279.4) (xy 34.29 279.4))
     (stroke (width 0) (type default))
   )
@@
     (stroke (width 0) (type default))
   )
-  (wire (pts (xy 396.24 218.44) (xy 396.24 223.52))
+  (wire (pts (xy 27.94 279.4) (xy 27.94 284.48))
     (stroke (width 0) (type default))
   )
@@
     (stroke (width 0) (type default))
   )
-  (wire (pts (xy 396.24 223.52) (xy 396.24 229.87))
+  (wire (pts (xy 27.94 284.48) (xy 27.94 290.83))
     (stroke (width 0) (type default))
   )
@@
     (stroke (width 0) (type default))
   )
-  (wire (pts (xy 402.59 208.28) (xy 396.24 208.28))
+  (wire (pts (xy 34.29 269.24) (xy 27.94 269.24))
     (stroke (width 0) (type default))
   )
@@
     (effects (font (size 1.5 1.5) (thickness 0.5994) bold) (justify left bottom))
   )
-  (text "For Metal Shield" (at 396.24 204.47 0)
+  (text "For Metal Shield" (at 27.94 265.43 0)
     (effects (font (size 1.27 1.27)) (justify left bottom))
   )
@@
     )
   )
-  (symbol (lib_id "Mechanical:MountingHole_Pad") (at 405.13 213.36 270) (unit 1)
-    (in_bom yes) (on_board yes) (dnp no) (fields_autoplaced)
-    (property "Reference" "SHLD-2" (at 408.94 212.725 90) (do_not_autoplace)
+  (symbol (lib_id "Mechanical:MountingHole_Pad") (at 36.83 274.32 270) (unit 1)
+    (in_bom no) (on_board yes) (dnp no) (fields_autoplaced)
+    (property "Reference" "SHLD-2" (at 40.64 273.685 90) (do_not_autoplace)
       (effects (font (size 1.27 1.27)) (justify left))
     )
-    (property "Value" "MountingHole_Pad" (at 408.94 212.725 90)
+    (property "Value" "MountingHole_Pad" (at 40.64 273.685 90)
       (effects (font (size 1.27 1.27)) (justify left) hide)
     )
-    (property "Footprint" "MountingHole:MountingHole_4.3mm_M4_ISO14580_Pad_TopBottom" (at 405.13 213.36 0)
+    (property "Footprint" "MountingHole:MountingHole_4.3mm_M4_ISO14580_Pad_TopBottom" (at 36.83 274.32 0)
       (effects (font (size 1.27 1.27)) hide)
     )
-    (property "Datasheet" "~" (at 405.13 213.36 0)
+    (property "Datasheet" "~" (at 36.83 274.32 0)
       (effects (font (size 1.27 1.27)) hide)
     )
@@
   )
   (symbol (lib_id "Mechanical:MountingHole_Pad") (at 34.29 163.83 270) (unit 1)
-    (in_bom yes) (on_board yes) (dnp no) (fields_autoplaced)
+    (in_bom no) (on_board yes) (dnp no) (fields_autoplaced)
     (property "Reference" "M_KSI1" (at 38.1 163.195 90) (do_not_autoplace)
       (effects (font (size 1.27 1.27)) (justify left))
@@
     )
   )
-  (symbol (lib_id "Mechanical:MountingHole_Pad") (at 405.13 208.28 270) (unit 1)
-    (in_bom yes) (on_board yes) (dnp no) (fields_autoplaced)
-    (property "Reference" "SHLD-1" (at 408.94 207.645 90) (do_not_autoplace)
+  (symbol (lib_id "Mechanical:MountingHole_Pad") (at 36.83 269.24 270) (unit 1)
+    (in_bom no) (on_board yes) (dnp no) (fields_autoplaced)
+    (property "Reference" "SHLD-1" (at 40.64 268.605 90) (do_not_autoplace)
       (effects (font (size 1.27 1.27)) (justify left))
     )
-    (property "Value" "MountingHole_Pad" (at 408.94 207.645 90)
+    (property "Value" "MountingHole_Pad" (at 40.64 268.605 90)
       (effects (font (size 1.27 1.27)) (justify left) hide)
     )
-    (property "Footprint" "MountingHole:MountingHole_4.3mm_M4_ISO14580_Pad_TopBottom" (at 405.13 208.28 0)
+    (property "Footprint" "MountingHole:MountingHole_4.3mm_M4_ISO14580_Pad_TopBottom" (at 36.83 269.24 0)
       (effects (font (size 1.27 1.27)) hide)
     )
-    (property "Datasheet" "~" (at 405.13 208.28 0)
+    (property "Datasheet" "~" (at 36.83 269.24 0)
       (effects (font (size 1.27 1.27)) hide)
     )
@@
   )
   (symbol (lib_id "Mechanical:MountingHole_Pad") (at 34.29 173.99 270) (unit 1)
-    (in_bom yes) (on_board yes) (dnp no) (fields_autoplaced)
+    (in_bom no) (on_board yes) (dnp no) (fields_autoplaced)
     (property "Reference" "M_KSI3" (at 38.1 173.355 90) (do_not_autoplace)
       (effects (font (size 1.27 1.27)) (justify left))
@@
     )
   )
-  (symbol (lib_id "Mechanical:MountingHole_Pad") (at 405.13 218.44 270) (unit 1)
-    (in_bom yes) (on_board yes) (dnp no) (fields_autoplaced)
-    (property "Reference" "SHLD-3" (at 408.94 217.805 90) (do_not_autoplace)
+  (symbol (lib_id "Mechanical:MountingHole_Pad") (at 36.83 279.4 270) (unit 1)
+    (in_bom no) (on_board yes) (dnp no) (fields_autoplaced)
+    (property "Reference" "SHLD-3" (at 40.64 278.765 90) (do_not_autoplace)
       (effects (font (size 1.27 1.27)) (justify left))
     )
-    (property "Value" "MountingHole_Pad" (at 408.94 217.805 90)
+    (property "Value" "MountingHole_Pad" (at 40.64 278.765 90)
       (effects (font (size 1.27 1.27)) (justify left) hide)
     )
-    (property "Footprint" "MountingHole:MountingHole_4.3mm_M4_ISO14580_Pad_TopBottom" (at 405.13 218.44 0)
+    (property "Footprint" "MountingHole:MountingHole_4.3mm_M4_ISO14580_Pad_TopBottom" (at 36.83 279.4 0)
       (effects (font (size 1.27 1.27)) hide)
     )
-    (property "Datasheet" "~" (at 405.13 218.44 0)
+    (property "Datasheet" "~" (at 36.83 279.4 0)
       (effects (font (size 1.27 1.27)) hide)
     )
@@
   )
   (symbol (lib_id "Mechanical:MountingHole_Pad") (at 34.29 179.07 270) (unit 1)
-    (in_bom yes) (on_board yes) (dnp no) (fields_autoplaced)
+    (in_bom no) (on_board yes) (dnp no) (fields_autoplaced)
     (property "Reference" "M_KSI4" (at 38.1 178.435 90) (do_not_autoplace)
       (effects (font (size 1.27 1.27)) (justify left))
@@
   )
   (symbol (lib_id "Mechanical:MountingHole_Pad") (at 34.29 168.91 270) (unit 1)
-    (in_bom yes) (on_board yes) (dnp no) (fields_autoplaced)
+    (in_bom no) (on_board yes) (dnp no) (fields_autoplaced)
     (property "Reference" "M_KSI2" (at 38.1 168.275 90) (do_not_autoplace)
       (effects (font (size 1.27 1.27)) (justify left))
@@
     )
   )
-  (symbol (lib_id "Mechanical:MountingHole_Pad") (at 405.13 223.52 270) (unit 1)
-    (in_bom yes) (on_board yes) (dnp no) (fields_autoplaced)
-    (property "Reference" "SHLD-4" (at 408.94 222.885 90) (do_not_autoplace)
+  (symbol (lib_id "Mechanical:MountingHole_Pad") (at 36.83 284.48 270) (unit 1)
+    (in_bom no) (on_board yes) (dnp no) (fields_autoplaced)
+    (property "Reference" "SHLD-4" (at 40.64 283.845 90) (do_not_autoplace)
       (effects (font (size 1.27 1.27)) (justify left))
     )
-    (property "Value" "MountingHole_Pad" (at 408.94 222.885 90)
+    (property "Value" "MountingHole_Pad" (at 40.64 283.845 90)
       (effects (font (size 1.27 1.27)) (justify left) hide)
     )
-    (property "Footprint" "MountingHole:MountingHole_4.3mm_M4_ISO14580_Pad_TopBottom" (at 405.13 223.52 0)
+    (property "Footprint" "MountingHole:MountingHole_4.3mm_M4_ISO14580_Pad_TopBottom" (at 36.83 284.48 0)
       (effects (font (size 1.27 1.27)) hide)
     )
-    (property "Datasheet" "~" (at 405.13 223.52 0)
+    (property "Datasheet" "~" (at 36.83 284.48 0)
       (effects (font (size 1.27 1.27)) hide)
     )
@@
     )
   )
-  (symbol (lib_id "power:GND") (at 396.24 229.87 0) (unit 1)
+  (symbol (lib_id "power:GND") (at 27.94 290.83 0) (unit 1)
     (in_bom yes) (on_board yes) (dnp no)
-    (property "Reference" "#PWR029" (at 396.24 236.22 0)
+    (property "Reference" "#PWR029" (at 27.94 297.18 0)
       (effects (font (size 1.27 1.27)) hide)
     )
-    (property "Value" "GND" (at 396.24 233.68 0)
+    (property "Value" "GND" (at 27.94 294.64 0)
       (effects (font (size 1.27 1.27)))
     )
-    (property "Footprint" "" (at 396.24 229.87 0)
+    (property "Footprint" "" (at 27.94 290.83 0)
       (effects (font (size 1.27 1.27)) hide)
     )
-    (property "Datasheet" "" (at 396.24 229.87 0)
+    (property "Datasheet" "" (at 27.94 290.83 0)
       (effects (font (size 1.27 1.27)) hide)
     )
@@
       (effects (font (size 1.27 1.27)) (justify left))
     )
-    (property "Value" "100" (at 63.5 210.82 0)
+    (property "Value" "300" (at 63.5 210.82 0)
       (effects (font (size 1.27 1.27)) (justify left))
     )
