File: hw/MK-KS.kicad_sch (KiCad schematic)
At the start: 69 parts, among them J1 USB-PWR, J10 LOOP RES, J3 MKOB-Serial, J4 MuKOB IF, J5 KEY/PDL, J8 LOOP PWR, J9 SNDR/KOB, Q1 2N3904, Q1 G01N20LE, Q8 2N3905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

Commit message: KSInf-MkIII: New  JA: Add terminal block
Parts:
- M_KSI1, M_KSI2, M_KSI3, M_KSI4, SHLD-1, SHLD-2, SHLD-3, SHLD-4: now left out of the parts list
