File: hw/MK-KS-MkIII.kicad_sch (KiCad schematic)
At the start: 86 parts, among them J1 MuKOB IF, J10 SNDR/KOB, J4 COMM-DCE-10, J5 RPi-GPIO40, J6 I2C Disp, J7 KEY-PADDLE, J8 LOOP PWR, J9 Loop Cur Limit, Q1 2N3904, Q1 G01N20LE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

Commit message: MK-IF-MKIII and JackAdapter PCBs produced.
Parts:
- removed Q1 (x2): 2N3904, Package_TO_SOT_SMD:SOT-23-3, symbol Transistor_BJT:2N3904
- removed R4 (x2): 20k, Resistor_SMD:R_0805_2012Metric_Pad1.20x1.40mm_HandSolder, symbol Device:R_US
- added C9: 0.1u, Capacitor_SMD:C_0603_1608Metric_Pad1.08x0.95mm_HandSolder, symbol Device:C
- added Q2, Q3: MMBT3904, Package_TO_SOT_SMD:SOT-23, symbol Transistor_BJT:MMBT3904
- added R4 (x2): 20k, Resistor_SMD:R_0805_2012Metric_Pad1.20x1.40mm_HandSolder, symbol Device:R_US
Connections:
- net +3.3V: now also R4.2, R4.2
- net BZ-: now also Q3.3 (C)
- net DASH-: now also R4.1
- net DOT-: now also R4.1
- net GND: now also C9.2, Q3.2 (E)
- net LOOP_STATE: now also C9.1
- net SLG: now also Q2.2 (E)
- net at LED1.1 (K): now also Q2.3 (C)
- net at R2.2: now also Q2.1 (B)
- net at R2.2: now also Q3.1 (B)
Other:
- note added: "+ EXTERNALLY POWERED"
- note added: "4-400 OHM SOUNDER / 4-8 OHM KOB"
- note added: "EXTERNALLY POWERED -"
- note added: "Extrnal - Not part of Interface Board"
- note added: "FOR EXTERNALLY POWERED LOOP JUMPER J2 (LOOP PWR)"
- note removed: "4-150 OHM SOUNDER / 4-8 OHM KOB"
- note removed: "Extrnal - Not part of MuKOB"
